Commit message: Some_changes_.yaml_files

File: diplom_folder/urdf/my_robot.urdf (robot description, URDF)
Before this commit: robot my_robot, 3 links, 2 joints
Joints:
- joint camera_joint: origin xyz=0.1 0 0.2 rpy=0 0 0 -> xyz=0.0 0 1.5 rpy=0 0 0

Commit message: did_something_done_map_tag

File: diplom_folder/urdf/my_robot.urdf (robot description, URDF)
Before this commit: robot my_robot, 3 links, 2 joints
Links:
- removed link default_cam
Joints:
- removed joint camera_alias

Commit message: FUCKING SHIIIIIIIT

File: diplom_folder/urdf/my_robot.urdf (robot description, URDF)
Before this commit: robot my_robot, 2 links, 1 joints
Joints:
- joint camera_joint: origin xyz=0.0 0 1.5 rpy=0 0 0 -> xyz=0.0 0 0.5 rpy=0 0 0

Commit message: Navigation_not_done_yet_but_good

File: diplom_folder/urdf/my_robot.urdf (robot description, URDF)
Before this commit: robot my_robot, 2 links, 1 joints
Joints:
- joint camera_joint: origin xyz=0.0 0 0.5 rpy=0 0 0 -> xyz=0.0 0 0.5 rpy=0 1.57 0
